Commit message: dummy normalforce from collision points working IPC dofs for objects and forces transport use pybullet to debug sensor output

File: sofa_example/mesh/digit.urdf (robot description, URDF)
Before this commit: robot digit, 1 links, 0 joints
Links:
- link baseLink: geometry collision mesh filename=digit_decimated.stl scale=1 1 1; visual mesh filename=digit_decimated.stl scale=1 1 1

Commit message: fix cam position change change scaling issue

File: sofa_example/mesh/digit.urdf (robot description, URDF)
Before this commit: robot digit, 1 links, 0 joints
Links:
- link baseLink: geometry collision mesh filename=digit_transformed2.stl scale=1 1 1; visual mesh filename=digit_transformed2.stl scale=1 1 1
